Commit message: new drone model

File: urdf.old/lidar_mapper_drone.urdf (robot description, URDF)
Before this commit: robot lidar_mapper_drone, 25 links, 24 joints
Links:
- removed link antenna_stick
- removed link back_holder_optical_flow
- removed link left_cover_H7
- removed link right_cover_H7
- added link antena-stick, mass 0.03440631866056707; collision mesh filename=package://lidar_mapper_visualiser/urdf/meshes/antena-stick.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 scale=0.001 0.001 0.001; visual mesh filename=package://lidar_mapper_visualiser/urdf/meshes/antena-stick.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 scale=0.001 0.001 0.001
- added link back_holder, mass 0.07190673375826725; collision mesh filename=package://lidar_mapper_visualiser/urdf/meshes/back_holder.s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 scale=0.001 0.001 0.001; visual mesh filename=package://lidar_mapper_visualiser/urdf/meshes/back_holder.s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 scale=0.001 0.001 0.001
- added link left_cover, mass 0.09341169364233115; collision mesh filename=package://lidar_mapper_visualiser/urdf/meshes/left_cover.stl scale=0.001 0.001 0.001; visual mesh filename=package://lidar_mapper_visualiser/urdf/meshes/left_cover.stl scale=0.001 0.001 0.001
- added link right_cover, mass 0.09251921869007904; collision mesh filename=package://lidar_mapper_visualiser/urdf/meshes/right_cover.s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 scale=0.001 0.001 0.001; visual mesh filename=package://lidar_mapper_visualiser/urdf/meshes/right_cover.s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 scale=0.001 0.001 0.001
Joints:
- removed joint back_holder_optical_flow_Rigid-26
- removed joint drone_base_Rigid-23
- removed joint drone_base_Rigid-24
- removed joint drone_base_Rigid-25
- added joint back_holder_Rigid-22: type fixed, parent back_holder, child antena-stick, origin xyz=0.0095 0.03197260999999999 -0.025 rpy=-0.7853981633974483 -3.283760281271351e-62 1.665064276623699e-31
- added joint drone_base_Rigid-1: type fixed, parent drone_base, child back_holder, origin xyz=-0.08741136368379873 -0.009500001275705983 -0.002500000000000517 rpy=-5.552470375841605e-17 -1.6098369382336299e-15 1.570796326794898
- added joint drone_base_Rigid-15: type fixed, parent drone_base, child left_cover, origin xyz=0.06899999631620117 -0.015700001275705776 -0.0025000000000005187 rpy=-5.552470375841605e-17 -1.6098369382336299e-15 1.570796326794898
- added joint drone_base_Rigid-16: type fixed, parent drone_base, child right_cover, origin xyz=0.06899999631620114 0.015699998724294152 -0.0025000000000004676 rpy=-5.552470375841605e-17 -1.6098369382336299e-15 1.570796326794898
