Commit message: working with ardupilot

File: urdf/lidar_mapper_drone.urdf (robot description, URDF)
Before this commit: robot lidar_mapper_drone, 24 links, 23 joints
Links:
- added link drone_base_link
Joints:
- added joint base_to_body_joint: type fixed, parent drone_base_link, child drone_base, origin xyz=0 0 0 rpy=3.14159 0 0
- joint ldlidar_link_joint: origin xyz=-0.0085 -0.033 -0.012 rpy=0 3.6652 1.5708 -> xyz=-0.0085 -0.033 -0.012 rpy=0.0 3.6652 1.5708

Commit message: sync scan messages

File: urdf/lidar_mapper_drone.urdf (robot description, URDF)
Before this commit: robot lidar_mapper_drone, 25 links, 24 joints
Links:
- added link 7_inch_CCW_1, mass 0.004466869702984176; collision mesh filename=package://lidar_mapper_visualiser/urdf/meshes/7_inch_CCW_1.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 scale=0.001 0.001 0.001; visual mesh filename=package://lidar_mapper_visualiser/urdf/meshes/7_inch_CCW_1.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 scale=0.001 0.001 0.001
- added link 7_inch_CCW_2, mass 0.004466869702984176; collision mesh filename=package://lidar_mapper_visualiser/urdf/meshes/7_inch_CCW_2.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 scale=0.001 0.001 0.001; visual mesh filename=package://lidar_mapper_visualiser/urdf/meshes/7_inch_CCW_2.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 scale=0.001 0.001 0.001
- added link 7_inch_CW_1, mass 0.004466869703094844; collision mesh filename=package://lidar_mapper_visualiser/urdf/meshes/7_inch_CW_1.s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 scale=0.001 0.001 0.001; visual mesh filename=package://lidar_mapper_visualiser/urdf/meshes/7_inch_CW_1.s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 scale=0.001 0.001 0.001
- added link 7_inch_CW_2, mass 0.004466869703094844; collision mesh filename=package://lidar_mapper_visualiser/urdf/meshes/7_inch_CW_2.s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 scale=0.001 0.001 0.001; visual mesh filename=package://lidar_mapper_visualiser/urdf/meshes/7_inch_CW_2.s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 scale=0.001 0.001 0.001
- link drone_base_link: mass None -> 0.001
- link ldlidar_link: mass None -> 0.001
Joints:
- added joint motor_rotor_1_Rigid-31: type fixed, parent motor_rotor_1, child 7_inch_CW_2, origin xyz=0.0 -0.006106199999999999 0.0 rpy=-1.9721522630525278e-31 1.7516230804059725e-46 -5.551115123127094e-17
- added joint motor_rotor_2_Rigid-30: type fixed, parent motor_rotor_2, child 7_inch_CW_1, origin xyz=-2.120000000012112e-06 -0.006106199999999999 1.3400000000096669e-06 rpy=1.1832913578315177e-30 2.189528850507736e-47 -5.551115123126314e-17
- added joint motor_rotor_3_Rigid-32: type fixed, parent motor_rotor_3, child 7_inch_CCW_1, origin xyz=-1.5400000000020952e-06 -0.006106199999999999 1.980000000010307e-06 rpy=-1.972152263052529e-31 7.888609052210118e-31 -5.263181352021438e-30
- added joint motor_rotor_4_Rigid-29: type fixed, parent motor_rotor_4, child 7_inch_CCW_2, origin xyz=-1.5400000000020952e-06 -0.006106199999999999 1.9799999999925432e-06 rpy=-9.860761315262645e-32 -3.94430452610506e-31 -1.1102230246252798e-16

Commit message: refined urdf file

File: urdf/lidar_mapper_drone.urdf (robot description, URDF)
Before this commit: robot lidar_mapper_drone, 24 links, 23 joints
Links:
- removed link antena-stick
- removed link back_holder
- removed link left_cover
- removed link right_cover
- added link 7_inch_CCW_1, mass 0.004466869702984176; collision mesh filename=package://lidar_mapper_visualiser/urdf/meshes/7_inch_CCW_1.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 scale=0.001 0.001 0.001; visual mesh filename=package://lidar_mapper_visualiser/urdf/meshes/7_inch_CCW_1.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 scale=0.001 0.001 0.001
- added link 7_inch_CCW_2, mass 0.004466869702984176; collision mesh filename=package://lidar_mapper_visualiser/urdf/meshes/7_inch_CCW_2.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 scale=0.001 0.001 0.001; visual mesh filename=package://lidar_mapper_visualiser/urdf/meshes/7_inch_CCW_2.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 scale=0.001 0.001 0.001
- added link 7_inch_CW_1, mass 0.004466869703094844; collision mesh filename=package://lidar_mapper_visualiser/urdf/meshes/7_inch_CW_1.s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 scale=0.001 0.001 0.001; visual mesh filename=package://lidar_mapper_visualiser/urdf/meshes/7_inch_CW_1.s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 scale=0.001 0.001 0.001
- added link 7_inch_CW_2, mass 0.004466869703094844; collision mesh filename=package://lidar_mapper_visualiser/urdf/meshes/7_inch_CW_2.s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 scale=0.001 0.001 0.001; visual mesh filename=package://lidar_mapper_visualiser/urdf/meshes/7_inch_CW_2.s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 scale=0.001 0.001 0.001
- added link antenna_stick, mass 0.03440631866056707; collision mesh filename=package://lidar_mapper_visualiser/urdf/meshes/antenna_stick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 scale=0.001 0.001 0.001; visual mesh filename=package://lidar_mapper_visualiser/urdf/meshes/antenna_stick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 scale=0.001 0.001 0.001
- added link back_holder_optical_flow, mass 0.0878096751327429; collision mesh filename=package://lidar_mapper_visualiser/urdf/meshes/back_holder_o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 scale=0.001 0.001 0.001; visual mesh filename=package://lidar_mapper_visualiser/urdf/meshes/back_holder_o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 scale=0.001 0.001 0.001
- added link drone_base_link, mass 0.001
- added link left_cover_H7, mass 0.09235027638883513; collision mesh filename=package://lidar_mapper_visualiser/urdf/meshes/left_cover_H7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 scale=0.001 0.001 0.001; visual mesh filename=package://lidar_mapper_visualiser/urdf/meshes/left_cover_H7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 scale=0.001 0.001 0.001
- added link right_cover_H7, mass 0.09341169301733705; collision mesh filename=package://lidar_mapper_visualiser/urdf/meshes/right_cover_H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 scale=0.001 0.001 0.001; visual mesh filename=package://lidar_mapper_visualiser/urdf/meshes/right_cover_H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 scale=0.001 0.001 0.001
- link ldlidar_link: mass None -> 0.001
Joints:
- removed joint back_holder_Rigid-22
- removed joint drone_base_Rigid-1
- removed joint drone_base_Rigid-15
- removed joint drone_base_Rigid-16
- added joint back_holder_optical_flow_Rigid-26: type fixed, parent back_holder_optical_flow, child antenna_stick, origin xyz=-0.009500000000000001 0.021173009999999996 -0.02625 rpy=-0.5235987755982986 -2.252140986350246e-62 1.1419711492581944e-31
- added joint base_to_body_joint: type fixed, parent drone_base_link, child drone_base, origin xyz=0 0 0 rpy=3.14159 0 0
- added joint drone_base_Rigid-23: type fixed, parent drone_base, child right_cover_H7, origin xyz=0.06899999631620114 0.015699998724294152 -0.0025000000000004676 rpy=-5.552470375841605e-17 -1.6098369382336299e-15 1.570796326794898
- added joint drone_base_Rigid-24: type fixed, parent drone_base, child left_cover_H7, origin xyz=0.06899999631620117 -0.015700001275705776 -0.0025000000000005187 rpy=-5.552470375841605e-17 -1.6098369382336299e-15 1.570796326794898
- added joint drone_base_Rigid-25: type fixed, parent drone_base, child back_holder_optical_flow, origin xyz=-0.08741136368379877 0.009499998724293976 -0.002500000000000486 rpy=-5.552470375841605e-17 -1.6098369382336299e-15 1.570796326794898
- added joint motor_rotor_1_Rigid-31: type fixed, parent motor_rotor_1, child 7_inch_CW_2, origin xyz=0.0 -0.006106199999999999 0.0 rpy=-1.9721522630525278e-31 1.7516230804059725e-46 -5.551115123127094e-17
- added joint motor_rotor_2_Rigid-30: type fixed, parent motor_rotor_2, child 7_inch_CW_1, origin xyz=-2.120000000012112e-06 -0.006106199999999999 1.3400000000096669e-06 rpy=1.1832913578315177e-30 2.189528850507736e-47 -5.551115123126314e-17
- added joint motor_rotor_3_Rigid-32: type fixed, parent motor_rotor_3, child 7_inch_CCW_1, origin xyz=-1.5400000000020952e-06 -0.006106199999999999 1.980000000010307e-06 rpy=-1.972152263052529e-31 7.888609052210118e-31 -5.263181352021438e-30
- added joint motor_rotor_4_Rigid-29: type fixed, parent motor_rotor_4, child 7_inch_CCW_2, origin xyz=-1.5400000000020952e-06 -0.006106199999999999 1.9799999999925432e-06 rpy=-9.860761315262645e-32 -3.94430452610506e-31 -1.1102230246252798e-16
- joint ldlidar_link_joint: origin xyz=-0.0085 -0.033 -0.012 rpy=0 3.6652 1.5708 -> xyz=-0.0085 -0.033 -0.012 rpy=0.0 3.6652 1.5708

Commit message: fix timings

File: urdf/lidar_mapper_drone.urdf (robot description, URDF)
Before this commit: robot lidar_mapper_drone, 29 links, 28 joints
Links:
- removed link ldlidar_link
Joints:
- removed joint ldlidar_link_joint

Commit message: add octomap

File: urdf/lidar_mapper_drone.urdf (robot description, URDF)
Before this commit: robot lidar_mapper_drone, 28 links, 27 joints
Links:
- removed link drone_base_link
- added link base_link, mass 0.001
Joints:
- joint base_to_body_joint: parent drone_base_link -> base_link

Commit message: add gps model

File: urdf/lidar_mapper_drone.urdf (robot description, URDF)
Before this commit: robot lidar_mapper_drone, 28 links, 27 joints
Links:
- added link SoloGood_M10, mass 0.0119703708; visual mesh filename=package://lidar_mapper_visualiser/urdf/meshes/SoloGood_M10.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 scale=0.001 0.001 0.001
Joints:
- added joint back_holder_optical_flow_Rigid-33: type fixed, parent back_holder_optical_flow, child SoloGood_M10, origin xyz=-0.009500000000000001 0.06584037000000001 -0.0275 rpy=-1.5707963267948966 1.893646573411915e-46 -9.601928861622976e-16

Commit message: change naming

File: urdf/lidar_mapper_drone.urdf (robot description, URDF)
Before this commit: robot lidar_mapper_drone, 29 links, 28 joints
Links:
- link 7_inch_CCW_1: geometry collision mesh filename=package://lidar_mapper_visualizer/urdf/meshes/7_inch_CCW_1.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 scale=0.001 0.001 0.001; visual mesh filename=package://lidar_mapper_visualizer/urdf/meshes/7_inch_CCW_1.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 scale=0.001 0.001 0.001
- link 7_inch_CCW_2: geometry collision mesh filename=package://lidar_mapper_visualizer/urdf/meshes/7_inch_CCW_2.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 scale=0.001 0.001 0.001; visual mesh filename=package://lidar_mapper_visualizer/urdf/meshes/7_inch_CCW_2.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 scale=0.001 0.001 0.001
- link 7_inch_CW_1: geometry collision mesh filename=package://lidar_mapper_visualizer/urdf/meshes/7_inch_CW_1.s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 scale=0.001 0.001 0.001; visual mesh filename=package://lidar_mapper_visualizer/urdf/meshes/7_inch_CW_1.s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 scale=0.001 0.001 0.001
- link 7_inch_CW_2: geometry collision mesh filename=package://lidar_mapper_visualizer/urdf/meshes/7_inch_CW_2.s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 scale=0.001 0.001 0.001; visual mesh filename=package://lidar_mapper_visualizer/urdf/meshes/7_inch_CW_2.s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 scale=0.001 0.001 0.001
- link CNHL_5S_2200MAH_LIPO: geometry collision mesh filename=package://lidar_mapper_visualizer/urdf/meshes/CNHL_5S_2200M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 scale=0.001 0.001 0.001; visual mesh filename=package://lidar_mapper_visualizer/urdf/meshes/CNHL_5S_2200M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 scale=0.001 0.001 0.001
- link SoloGood_M10: geometry visual mesh filename=package://lidar_mapper_visualizer/urdf/meshes/SoloGood_M10.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 scale=0.001 0.001 0.001
- link antenna_stick: geometry collision mesh filename=package://lidar_mapper_visualizer/urdf/meshes/antenna_stick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 scale=0.001 0.001 0.001; visual mesh filename=package://lidar_mapper_visualizer/urdf/meshes/antenna_stick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 scale=0.001 0.001 0.001
- link back_holder_optical_flow: geometry collision mesh filename=package://lidar_mapper_visualizer/urdf/meshes/back_holder_o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 scale=0.001 0.001 0.001; visual mesh filename=package://lidar_mapper_visualizer/urdf/meshes/back_holder_o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 scale=0.001 0.001 0.001
- link camera_1800TVL: geometry collision mesh filename=package://lidar_mapper_visualizer/urdf/meshes/camera_1800TV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 scale=0.001 0.001 0.001; visual mesh filename=package://lidar_mapper_visualizer/urdf/meshes/camera_1800TV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 scale=0.001 0.001 0.001
- link damper_1: geometry collision mesh filename=package://lidar_mapper_visualizer/urdf/meshes/damper_1.stl scale=0.001 0.001 0.001; visual mesh filename=package://lidar_mapper_visualizer/urdf/meshes/damper_1.stl scale=0.001 0.001 0.001
- link damper_2: geometry collision mesh filename=package://lidar_mapper_visualizer/urdf/meshes/damper_2.stl scale=0.001 0.001 0.001; visual mesh filename=package://lidar_mapper_visualizer/urdf/meshes/damper_2.stl scale=0.001 0.001 0.001
- link damper_3: geometry collision mesh filename=package://lidar_mapper_visualizer/urdf/meshes/damper_3.stl scale=0.001 0.001 0.001; visual mesh filename=package://lidar_mapper_visualizer/urdf/meshes/damper_3.stl scale=0.001 0.001 0.001
- link drone_base: geometry collision mesh filename=package://lidar_mapper_visualizer/urdf/meshes/drone_base.stl scale=0.001 0.001 0.001; visual mesh filename=package://lidar_mapper_visualizer/urdf/meshes/drone_base.stl scale=0.001 0.001 0.001
- link ldlidar_base: geometry collision mesh filename=package://lidar_mapper_visualizer/urdf/meshes/LD19.stl scale=0.001 0.001 0.001; visual mesh filename=package://lidar_mapper_visualizer/urdf/meshes/LD19.stl scale=0.001 0.001 0.001
- link left_cover_H7: geometry collision mesh filename=package://lidar_mapper_visualizer/urdf/meshes/left_cover_H7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 scale=0.001 0.001 0.001; visual mesh filename=package://lidar_mapper_visualizer/urdf/meshes/left_cover_H7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 scale=0.001 0.001 0.001
- link lidar_mount_30deg: geometry collision mesh filename=package://lidar_mapper_visualizer/urdf/meshes/lidar_mount_3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 scale=0.001 0.001 0.001; visual mesh filename=package://lidar_mapper_visualizer/urdf/meshes/lidar_mount_3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 scale=0.001 0.001 0.001
- link motor_rotor_1: geometry collision mesh filename=package://lidar_mapper_visualizer/urdf/meshes/motor_rotor_1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 scale=0.001 0.001 0.001; visual mesh filename=package://lidar_mapper_visualizer/urdf/meshes/motor_rotor_1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 scale=0.001 0.001 0.001
- link motor_rotor_2: geometry collision mesh filename=package://lidar_mapper_visualizer/urdf/meshes/motor_rotor_2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 scale=0.001 0.001 0.001; visual mesh filename=package://lidar_mapper_visualizer/urdf/meshes/motor_rotor_2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 scale=0.001 0.001 0.001
- link motor_rotor_3: geometry collision mesh filename=package://lidar_mapper_visualizer/urdf/meshes/motor_rotor_3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 scale=0.001 0.001 0.001; visual mesh filename=package://lidar_mapper_visualizer/urdf/meshes/motor_rotor_3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 scale=0.001 0.001 0.001
- link motor_rotor_4: geometry collision mesh filename=package://lidar_mapper_visualizer/urdf/meshes/motor_rotor_4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 scale=0.001 0.001 0.001; visual mesh filename=package://lidar_mapper_visualizer/urdf/meshes/motor_rotor_4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 scale=0.001 0.001 0.001
- link motor_stator_1: geometry collision mesh filename=package://lidar_mapper_visualizer/urdf/meshes/motor_stator_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 scale=0.001 0.001 0.001; visual mesh filename=package://lidar_mapper_visualizer/urdf/meshes/motor_stator_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 scale=0.001 0.001 0.001
- link motor_stator_2: geometry collision mesh filename=package://lidar_mapper_visualizer/urdf/meshes/motor_stator_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 scale=0.001 0.001 0.001; visual mesh filename=package://lidar_mapper_visualizer/urdf/meshes/motor_stator_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 scale=0.001 0.001 0.001
- link motor_stator_3: geometry collision mesh filename=package://lidar_mapper_visualizer/urdf/meshes/motor_stator_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 scale=0.001 0.001 0.001; visual mesh filename=package://lidar_mapper_visualizer/urdf/meshes/motor_stator_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 scale=0.001 0.001 0.001
- link motor_stator_4: geometry collision mesh filename=package://lidar_mapper_visualizer/urdf/meshes/motor_stator_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 scale=0.001 0.001 0.001; visual mesh filename=package://lidar_mapper_visualizer/urdf/meshes/motor_stator_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 scale=0.001 0.001 0.001
- link orangepi: geometry collision mesh filename=package://lidar_mapper_visualizer/urdf/meshes/orangepi.stl scale=0.001 0.001 0.001; visual mesh filename=package://lidar_mapper_visualizer/urdf/meshes/orangepi.stl scale=0.001 0.001 0.001
- link raspbox: geometry collision mesh filename=package://lidar_mapper_visualizer/urdf/meshes/raspbox.stl scale=0.001 0.001 0.001; visual mesh filename=package://lidar_mapper_visualizer/urdf/meshes/raspbox.stl scale=0.001 0.001 0.001
- link raspbox_top: geometry collision mesh filename=package://lidar_mapper_visualizer/urdf/meshes/raspbox_top.s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 scale=0.001 0.001 0.001; visual mesh filename=package://lidar_mapper_visualizer/urdf/meshes/raspbox_top.s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 scale=0.001 0.001 0.001
- link right_cover_H7: geometry collision mesh filename=package://lidar_mapper_visualizer/urdf/meshes/right_cover_H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 scale=0.001 0.001 0.001; visual mesh filename=package://lidar_mapper_visualizer/urdf/meshes/right_cover_H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 scale=0.001 0.001 0.001
